File: Prototypes/Arduino-UNO-Proto-Sheild/Arduino-UNO-Sheild.brd (EAGLE design)
At the start: 160 x 100 mm, 1 part, among them J1 ARDUINO_R3_SHIELD

Commit message: Fixes
Parts:
- added R1, R2, R3, R4, R5, R6, R7, R8: 10k, SparkFun-Passives:AXIAL-0.3-KIT
- added SW1: (no value), SparkFun-Electromechanical:DIPSWITCH-08
- added U$1: CATALEX-MICROSD-BREAKOUT, Modules:CATALEX-MICROSD-BREAKOUT
- added U$2: MPU-9250-BREAKOUT, Modules:MPU-9250-BREAKOUT
Connections:
- new net N$1: J1.A4, U$2.SDA
- new net N$10: J1.D9, R1.P$1, SW1.8
- new net N$11: J1.D8, R2.P$1, SW1.7
- new net N$12: J1.D7, R3.P$1, SW1.6
- new net N$13: J1.D6, R4.P$1, SW1.5
- new net N$14: J1.D5, R5.P$1, SW1.4
- new net N$15: J1.D4, R6.P$1, SW1.3
- new net N$16: J1.D3, R7.P$1, SW1.2
- new net N$17: J1.D2, R8.P$1, SW1.1
- new net N$18: J1.5V, SW1.10, SW1.11, SW1.12, SW1.13, SW1.14, SW1.15, SW1.16, SW1.9, U$1.VCC
- new net N$2: J1.A5, U$2.SCL
- new net N$20: J1.GND@2, R1.P$2, R2.P$2, R3.P$2, R4.P$2, R5.P$2, R6.P$2, R7.P$2, R8.P$2, U$1.GND
- new net N$3: J1.3.3V, U$2.AD0, U$2.VCC
- new net N$4: J1.GND@0, U$2.GND
- new net N$6: J1.D10, U$1.CS
- new net N$7: J1.D13, U$1.SCK
- new net N$8: J1.D11, U$1.MOSI
- new net N$9: J1.D12, U$1.MISO
Routing:
- net N$20: track 0.00 -> 165.9 mm
- net N$18: track 0.00 -> 66.1 mm
- net N$3: track 0.00 -> 65.0 mm
- net N$7: track 0.00 -> 55.5 mm
- net N$9: track 0.00 -> 46.1 mm
- net N$8: track 0.00 -> 46.1 mm
- net N$6: track 0.00 -> 45.1 mm
- net N$2: track 0.00 -> 24.4 mm
- net N$10: track 0.00 -> 21.5 mm
- net N$11: track 0.00 -> 20.4 mm
- net N$17: track 0.00 -> 19.9 mm
- net N$16: track 0.00 -> 18.8 mm
- net N$15: track 0.00 -> 18.8 mm
- net N$14: track 0.00 -> 18.8 mm
- net N$13: track 0.00 -> 17.8 mm
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
Commit message: Fixes
Routing:
- net N$3: track 65.0 -> 66.0 mm
- net N$2: track 24.4 -> 25.2 mm
Other:
- board size 160 x 100 mm -> 57.1 x 59.7 mm
Changed lines of the file:
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@@
 <layer number="18" name="Vias" color="2" fill="1" visible="yes" active="yes"/>
 <layer number="19" name="Unrouted" color="6" fill="1" visible="yes" active="yes"/>
-<layer number="20" name="Dimension" color="15" fill="1" visible="no" active="yes"/>
+<layer number="20" name="Dimension" color="15" fill="1" visible="yes" active="yes"/>
 <layer number="21" name="tPlace" color="7" fill="1" visible="yes" active="yes"/>
 <layer number="22" name="bPlace" color="7" fill="1" visible="yes" active="yes"/>
@@
 <layer number="50" name="dxf" color="7" fill="1" visible="no" active="no"/>
 <layer number="51" name="tDocu" color="7" fill="1" visible="yes" active="yes"/>
-<layer number="52" name="bDocu" color="7" fill="1" visible="yes" active="yes"/>
+<layer number="52" name="bDocu" color="7" fill="1" visible="no" active="yes"/>
 <layer number="53" name="tGND_GNDA" color="7" fill="9" visible="no" active="no"/>
 <layer number="54" name="bGND_GNDA" color="1" fill="9" visible="no" active="no"/>
@@
 <layer number="105" name="tPlate" color="7" fill="1" visible="yes" active="yes"/>
 <layer number="106" name="bPlate" color="7" fill="1" visible="yes" active="yes"/>
-<layer number="107" name="Crop" color="7" fill="1" visible="yes" active="yes"/>
+<layer number="107" name="Crop" color="7" fill="1" visible="no" active="yes"/>
 <layer number="108" name="tplace-old" color="10" fill="1" visible="yes" active="yes"/>
 <layer number="109" name="ref-old" color="11" fill="1" visible="yes" active="yes"/>
@@
 <board>
 <plain>
-<wire x1="0" y1="0" x2="160" y2="0" width="0" layer="20"/>
-<wire x1="160" y1="0" x2="160" y2="100" width="0" layer="20"/>
-<wire x1="160" y1="100" x2="0" y2="100" width="0" layer="20"/>
-<wire x1="0" y1="100" x2="0" y2="0" width="0" layer="20"/>
+<wire x1="-68.58" y1="74.6" x2="-68.58" y2="20.526090625" width="0" layer="20"/>
+<wire x1="-68.58" y1="20.526090625" x2="-64.563909375" y2="16.51" width="0" layer="20"/>
+<wire x1="-64.563909375" y1="16.51" x2="-14.280915625" y2="16.51" width="0" layer="20"/>
+<wire x1="-14.280915625" y1="16.51" x2="-11.45" y2="19.340915625" width="0" layer="20"/>
+<wire x1="-11.45" y1="19.340915625" x2="-11.45" y2="72.06" width="0" layer="20"/>
+<wire x1="-11.45" y1="72.06" x2="-11.43" y2="72.39" width="0" layer="20"/>
+<wire x1="-11.43" y1="72.39" x2="-15.24" y2="76.2" width="0" layer="20"/>
+<wire x1="-15.24" y1="76.2" x2="-52.07" y2="76.2" width="0" layer="20"/>
+<wire x1="-52.07" y1="76.2" x2="-53.67" y2="74.6" width="0" layer="20"/>
+<wire x1="-53.67" y1="74.6" x2="-68.58" y2="74.6" width="0" layer="20"/>
 </plain>
 <attributes>
@@
 <contactref element="J1" pad="A5"/>
 <wire x1="-22.86" y1="53.34" x2="-20.32" y2="55.88" width="0.6096" layer="16"/>
-<wire x1="-20.32" y1="55.88" x2="-15.24" y2="55.88" width="0.6096" layer="16"/>
-<wire x1="-15.24" y1="55.88" x2="-15.24" y2="69.85" width="0.6096" layer="16"/>
-<wire x1="-15.24" y1="69.85" x2="-16.51" y2="71.12" width="0.6096" layer="16"/>
+<wire x1="-20.32" y1="55.88" x2="-15.76605" y2="55.88" width="0.6096" layer="16"/>
+<wire x1="-15.76605" y1="55.88" x2="-13.97" y2="57.67605" width="0.6096" layer="16"/>
+<wire x1="-13.97" y1="57.67605" x2="-13.97" y2="68.58" width="0.6096" layer="16"/>
+<wire x1="-13.97" y1="68.58" x2="-16.51" y2="71.12" width="0.6096" layer="16"/>
 </signal>
 <signal name="N$3">
@@
 <wire x1="-25.4" y1="50.8" x2="-25.4" y2="60.96" width="0.6096" layer="16"/>
 <wire x1="-25.4" y1="60.96" x2="-22.86" y2="63.5" width="0.6096" layer="16"/>
-<wire x1="-16.51" y1="43.18" x2="-13.97" y2="45.72" width="0.6096" layer="16"/>
-<wire x1="-13.97" y1="45.72" x2="-13.97" y2="71.12" width="0.6096" layer="16"/>
-<wire x1="-13.97" y1="71.12" x2="-16.51" y2="73.66" width="0.6096" layer="16"/>
+<wire x1="-16.51" y1="43.18" x2="-12.7" y2="46.99" width="0.6096" layer="16"/>
+<wire x1="-12.7" y1="46.99" x2="-12.7" y2="69.85" width="0.6096" layer="16"/>
+<wire x1="-12.7" y1="69.85" x2="-16.51" y2="73.66" width="0.6096" layer="16"/>
 <wire x1="-16.51" y1="73.66" x2="-20.32" y2="73.66" width="0.6096" layer="16"/>
 <wire x1="-20.32" y1="73.66" x2="-21.59" y2="72.39" width="0.6096" layer="16"/>
